File: schematics/8-bit-cpu/clock_module.sch (KiCad schematic (older format))
At the start: 21 parts

Commit message: Added ALU, Accumulator and HL register schematics
Parts:
- added U? (x2): NE556, symbol Timer:NE556
- added U?: NE555, symbol Timer:NE555
- added U? (x4): 74LS00, symbol 74xx:74LS00
- C? (x5): symbol Clock-eagle-import:C5_3 -> 8-bit-cpu-rescue:C5_3-Clock-eagle-import
- IC? (x3): symbol Clock-eagle-import:DIL14 -> 8-bit-cpu-rescue:DIL14-Clock-eagle-import
- IC?: symbol Clock-eagle-import:DIL8 -> 8-bit-cpu-rescue:DIL8-Clock-eagle-import
- JP?: symbol Clock-eagle-import:JP1E -> 8-bit-cpu-rescue:JP1E-Clock-eagle-import
- LED?: symbol Clock-eagle-import:LED_ELD260 -> 8-bit-cpu-rescue:LED_ELD260-Clock-eagle-import
- R? (x7): symbol Clock-eagle-import:R0204_7 -> 8-bit-cpu-rescue:R0204_7-Clock-eagle-import
- S? (x2): symbol Clock-eagle-import:TL36PO -> 8-bit-cpu-rescue:TL36PO-Clock-eagle-import
- S?: symbol Clock-eagle-import:10-XX -> 8-bit-cpu-rescue:10-XX-Clock-eagle-import
Changed lines of the file:
@@
 EESchema Schematic File Version 4
 LIBS:8-bit-cpu-cache
-LIBS:Clock-cache
 EELAYER 26 0
 EELAYER END
 $Descr A4 8268 11693 portrait
 encoding utf-8
-Sheet 3 3
+Sheet 3 6
 Title ""
 Date ""
@@
 	3950 8100 3850 8100
 Wire Wire Line
-	3850 8100 3850 8400
-Wire Wire Line
-	3850 8400 4650 8400
-Wire Wire Line
-	4650 8400 4650 8000
+	3850 8500 4650 8500
 Wire Wire Line
 	4650 8000 4550 8000
@@
 Connection ~ 5550 2700
 $Comp
-L Clock-eagle-import:DIL14 IC?
+L 8-bit-cpu-rescue:DIL14-Clock-eagle-import IC?
 U 1 0 4268546C
 P 4250 3200
@@
 $EndComp
 $Comp
-L Clock-eagle-import:DIL14 IC?
+L 8-bit-cpu-rescue:DIL14-Clock-eagle-import IC?
 U 1 0 8113A942
 P 4250 7000
@@
 $EndComp
 $Comp
-L Clock-eagle-import:DIL14 IC?
+L 8-bit-cpu-rescue:DIL14-Clock-eagle-import IC?
 U 1 0 92DB5C2D
 P 4250 8000
@@
 $EndComp
 $Comp
-L Clock-eagle-import:DIL8 IC?
+L 8-bit-cpu-rescue:DIL8-Clock-eagle-import IC?
 U 1 0 0E69B6DF
 P 4250 6000
@@
 $EndComp
 $Comp
-L Clock-eagle-import:C5_3 C?
+L 8-bit-cpu-rescue:C5_3-Clock-eagle-import C?
 U 1 0 C8E3AF05
 P 4750 3200
@@
 $EndComp
 $Comp
-L Clock-eagle-import:10-XX S?
+L 8-bit-cpu-rescue:10-XX-Clock-eagle-import S?
 U 1 0 788C9994
 P 4250 4300
+AR Path="/788C9994" Ref="S?"  Part="1"
+AR Path="/5C215D87/788C9994" Ref="S?"  Part="1"
 F 0 "S?" V 4000 4200 59  0000 L BNN
 F 1 "10-XX" V 4100 4425 59  0000 L BNN
@@
 $EndComp
 $Comp
-L Clock-eagle-import:C5_3 C?
+L 8-bit-cpu-rescue:C5_3-Clock-eagle-import C?
 U 1 0 2DB567F5
 P 5050 6200
@@
 $EndComp
 $Comp
-L Clock-eagle-import:TL36PO S?
+L 8-bit-cpu-rescue:TL36PO-Clock-eagle-import S?
 U 1 0 F9B5905E
 P 3550 4300
@@
 $EndComp
 $Comp
-L Clock-eagle-import:TL36PO S?
+L 8-bit-cpu-rescue:TL36PO-Clock-eagle-import S?
 U 1 0 638E9151
 P 3450 5400
@@
 $EndComp
 $Comp
-L Clock-eagle-import:C5_3 C?
+L 8-bit-cpu-rescue:C5_3-Clock-eagle-import C?
 U 1 0 504B87AF
 P 3250 4000
@@
 $EndComp
 $Comp
-L Clock-eagle-import:C5_3 C?
+L 8-bit-cpu-rescue:C5_3-Clock-eagle-import C?
 U 1 0 487BCAB4
 P 3250 4600
@@
 $EndComp
 $Comp
-L Clock-eagle-import:LED_ELD260 LED?
+L 8-bit-cpu-rescue:LED_ELD260-Clock-eagle-import LED?
 U 1 0 7DC8C285
 P 3250 6800
@@
 $EndComp
 $Comp
-L Clock-eagle-import:R0204_7 R?
+L 8-bit-cpu-rescue:R0204_7-Clock-eagle-import R?
 U 1 0 B13F4994
 P 5150 4300
@@
 $EndComp
 $Comp
-L Clock-eagle-import:R0204_7 R?
+L 8-bit-cpu-rescue:R0204_7-Clock-eagle-import R?
 U 1 0 A04F324A
 P 5250 3100
@@
 $EndComp
 $Comp
-L Clock-eagle-import:R0204_7 R?
+L 8-bit-cpu-rescue:R0204_7-Clock-eagle-import R?
 U 1 0 DDF01354
 P 3050 2700
@@
 $EndComp
 $Comp
-L Clock-eagle-import:R0204_7 R?
+L 8-bit-cpu-rescue:R0204_7-Clock-eagle-import R?
 U 1 0 151DF089
 P 3050 3100
@@
 $EndComp
 $Comp
-L Clock-eagle-import:R0204_7 R?
+L 8-bit-cpu-rescue:R0204_7-Clock-eagle-import R?
 U 1 0 4373A00B
 P 5150 5300
@@
 $EndComp
 $Comp
-L Clock-eagle-import:R0204_7 R?
+L 8-bit-cpu-rescue:R0204_7-Clock-eagle-import R?
 U 1 0 9270C831
 P 5150 5700
@@
 $EndComp
 $Comp
-L Clock-eagle-import:R0204_7 R?
+L 8-bit-cpu-rescue:R0204_7-Clock-eagle-import R?
 U 1 0 5DDD930F
 P 3450 7200
@@
 $EndComp
 $Comp
-L Clock-eagle-import:GND #SUPPLY?
+L 8-bit-cpu-rescue:GND-Clock-eagle-import #SUPPLY?
 U 1 0 F54A36B8
 P 5850 2800
@@
 $EndComp
 $Comp
-L Clock-eagle-import:JP1E JP?
+L 8-bit-cpu-rescue:JP1E-Clock-eagle-import JP?
 U 1 0 0B60073D
 P 5450 2200
@@
 $EndComp
 $Comp
-L Clock-eagle-import:VCC #P+?
+L 8-bit-cpu-rescue:VCC-Clock-eagle-import #P+?
 U 1 0 6A081B6E
 P 5250 2100
@@
 $EndComp
 $Comp
-L Clock-eagle-import:C5_3 C?
+L 8-bit-cpu-rescue:C5_3-Clock-eagle-import C?
 U 1 0 8E04CE4C
 P 5350 2700
@@
 Wire Wire Line
 	3750 7200 3650 7200
+Wire Wire Line
+	3850 8100 3850 8500
+Wire Wire Line
+	4650 8000 4650 8500
+$Comp
+L Timer:NE556 U?
+U 1 1 5C234B1F
+P 3250 1350
+F 0 "U?" H 3250 1928 50  0000 C CNN
+F 1 "NE556" H 3250 1837 50  0000 C CNN
+F 2 "" H 3250 1350 50  0001 C CNN
+F 3 "http://www.ti.com/lit/ds/symlink/ne556.pdf" H 3250 1350 50  0001 C CNN
+	1    3250 1350
+	1    0    0    -1
+$EndComp
+$Comp
+L Timer:NE556 U?
+U 2 1 5C234EB0
+P 4350 1350
+F 0 "U?" H 4350 1928 50  0000 C CNN
+F 1 "NE556" H 4350 1837 50  0000 C CNN
+F 2 "" H 4350 1350 50  0001 C CNN
+F 3 "http://www.ti.com/lit/ds/symlink/ne556.pdf" H 4350 1350 50  0001 C CNN
+	2    4350 1350
+	1    0    0    -1
+$EndComp
+$Comp
+L Timer:NE555 U?
+U 1 1 5C235618
+P 2150 1350
+F 0 "U?" H 2150 1928 50  0000 C CNN
+F 1 "NE555" H 2150 1837 50  0000 C CNN
+F 2 "" H 2150 1350 50  0001 C CNN
+F 3 "http://www.ti.com/lit/ds/symlink/ne555.pdf" H 2150 1350 50  0001 C CNN
+	1    2150 1350
+	1    0    0    -1
+$EndComp
+$Comp
+L 74xx:74LS00 U?
+U 1 1 5C235DC8
+P 2150 7750
+F 0 "U?" H 2150 8075 50  0000 C CNN
+F 1 "74LS00" H 2150 7984 50  0000 C CNN
+F 2 "" H 2150 7750 50  0001 C CNN
+F 3 "http://www.ti.com/lit/gpn/sn74ls00" H 2150 7750 50  0001 C CNN
+	1    2150 7750
+	1    0    0    -1
+$EndComp
+$Comp
+L 74xx:74LS00 U?
+U 2 1 5C235EFE
+P 2150 8300
+F 0 "U?" H 2150 8625 50  0000 C CNN
+F 1 "74LS00" H 2150 8534 50  0000 C CNN
+F 2 "" H 2150 8300 50  0001 C CNN
+F 3 "http://www.ti.com/lit/gpn/sn74ls00" H 2150 8300 50  0001 C CNN
+	2    2150 8300
+	1    0    0    -1
+$EndComp
+$Comp
+L 74xx:74LS00 U?
+U 3 1 5C23AA09
+P 2150 8850
+F 0 "U?" H 2150 9175 50  0000 C CNN
+F 1 "74LS00" H 2150 9084 50  0000 C CNN
+F 2 "" H 2150 8850 50  0001 C CNN
+F 3 "http://www.ti.com/lit/gpn/sn74ls00" H 2150 8850 50  0001 C CNN
+	3    2150 8850
+	1    0    0    -1
+$EndComp
+$Comp
+L 74xx:74LS00 U?
+U 4 1 5C23AC3F
+P 2150 9400
+F 0 "U?" H 2150 9725 50  0000 C CNN
+F 1 "74LS00" H 2150 9634 50  0000 C CNN
+F 2 "" H 2150 9400 50  0001 C CNN
+F 3 "http://www.ti.com/lit/gpn/sn74ls00" H 2150 9400 50  0001 C CNN
+	4    2150 9400
+	1    0    0    -1
+$EndComp
 $EndSCHEMATC
